File: Hardware/SCHEMATIC.sch (EAGLE design)
At the start: 105 parts, among them IC1 BQ25180YBGR, IC2 DRV2605YZFR, IC3 BMA421, IC9 RT6160AWSC, J1 503480-2400, J2 TC2030-IDC, J4 KH-TYPE-C-16P_KH-TYPE-C-16P, Q1 DMG2305UX-7, Q3 SI1308EDL-T1-GE3, U1 NRF52840_QF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

Commit message: Upload final release: Hardware, Manufacturing and 3D files
Parts:
- C1-EP-DR, C24, C25, C33, C39: device InkTime_v5:NORDIC_NRF_3_CAPACITOR_0201_L -> InkTime_v5:NORDIC_NRF_3_CAPACITOR_0402_L
- D2, D4, D5: value ESP32_C6_LIBRARY_5_MBR0530 -> MBR0530
Connections:
- removed net N$5: C33.1
- net 3V3: now also C33.1
